Commit message: add ground

File: src/abot_description/urdf/abot.xacro (robot description, xacro)
@@ -4,4 +4,5 @@
 	<!-- Matherials -->
 	<xacro:include filename="$(find abot_description)/urdf/abot_matherials.xacro" />
+	<xacro:property name="clearance" value="0.018" />
 	<!-- abot_base -->
 	<link name="abot_base">
@@ -39,4 +40,19 @@
 		<child link="abot_base" />
 	</joint>
+	<!-- base_footprint -->
+	<link name="base_footprint">
+		<visual>
+			<origin xyz="0 0 0" rpy="0 0 0" />
+			<geometry>
+				<cylinder length="0.001" radius="0.010" />
+			</geometry>
+			<material name="Blue" />
+		</visual>
+	</link>
+	<joint name="base_footprint_to_base_link" type="fixed">
+		<origin xyz="0 0 ${clearance}" rpy="0 0 0" />
+		<parent link="base_footprint" />
+		<child link="base_link" />
+	</joint>
 	<!-- Wheels -->
 	<xacro:include filename="$(find abot_description)/urdf/abot_left_wheel.xacro" />
